Commit message: [Beetle_hyper][URDF]Change the urdf and mesh file of quad into Beetle_hyper version

File: robots/gimbalrotor/urdf/quad/gimbalrotor.urdf.xacro (robot description, xacro)
@@ -23,14 +23,14 @@
     <link name="base_link">
       <inertial>
-        <origin xyz="0.0 0.0 0.0165" rpy="0 0 0"/>
-        <mass value="0.1753"/>
-        <inertia
-            ixx="0.0004" iyy="0.0004" izz="0.0008"
-            ixy="0.00000" ixz="0.0000" iyz="0.00000"/>
-      </inertial>
-      <visual>
-        <origin xyz="0 0 -0.0165" rpy="0 0 0"/>
-        <geometry>
-          <mesh filename="package://gimbalrotor/urdf/quad/mesh/base_link.STL"/>
+        <origin xyz="0.0257171 0.0007358  0.0813823" rpy="0 0 0"/>
+        <mass value="2.8200834"/>
+        <inertia
+            ixx="0.0679394" iyy="0.1142367" izz="0.1213159"
+            ixy="-0.0001621" ixz="0.00612466" iyz="0.0000964"/>
+      </inertial>
+      <visual>
+        <origin xyz="0 0 0" rpy="0 0 3.141592"/>
+        <geometry>
+          <mesh filename="package://gimbalrotor/urdf/quad/mesh/base_link_hyper.dae"/>
         </geometry>
       </visual>
@@ -72,5 +72,5 @@
         <origin xyz="0 0 0" rpy="0 0 0"/>
         <geometry>
-          <mesh filename="package://gimbalrotor/urdf/quad/mesh/rotor_arm.STL"/>
+          <mesh filename="package://gimbalrotor/urdf/quad/mesh/rotor_arm.dae"/>
         </geometry>
       </visual>
@@ -100,5 +100,5 @@
         <origin xyz="0 0 0" rpy="0 0 0"/>
         <geometry>
-          <mesh filename="package://gimbalrotor/urdf/quad/mesh/rotor_arm.STL"/>
+          <mesh filename="package://gimbalrotor/urdf/quad/mesh/rotor_arm.dae"/>
         </geometry>
       </visual>
@@ -128,5 +128,5 @@
         <origin xyz="0 0 0" rpy="0 0 0"/>
         <geometry>
-          <mesh filename="package://gimbalrotor/urdf/quad/mesh/rotor_arm.STL"/>
+          <mesh filename="package://gimbalrotor/urdf/quad/mesh/rotor_arm.dae"/>
         </geometry>
       </visual>
@@ -156,5 +156,5 @@
         <origin xyz="0 0 0" rpy="0 0 0"/>
         <geometry>
-          <mesh filename="package://gimbalrotor/urdf/quad/mesh/rotor_arm.STL"/>
+          <mesh filename="package://gimbalrotor/urdf/quad/mesh/rotor_arm.dae"/>
         </geometry>
       </visual>
@@ -194,5 +194,5 @@
         <origin xyz="0 0 0" rpy="0 0 0"/>
         <geometry>
-          <mesh filename="package://gimbalrotor/urdf/quad/mesh/rotor_module.STL"/>
+          <mesh filename="package://gimbalrotor/urdf/quad/mesh/rotor_module.dae"/>
         </geometry>
       </visual>

Commit message: [Beetle_hyper][URDF]Finised the adjustment of urdf

File: robots/gimbalrotor/urdf/quad/gimbalrotor.urdf.xacro (robot description, xacro)
@@ -36,7 +36,7 @@
       </visual>
       <collision>
-        <origin xyz="0 0 0" rpy="0 0 0"/>
-        <geometry>
-          <box size="0.25 0.25 0.035"/>
+        <origin xyz="0 0 0.053" rpy="0 0 0"/>
+        <geometry>
+          <box size="0.52 0.52 0.241"/>
         </geometry>
       </collision>
@@ -59,117 +59,47 @@
       <axis xyz="0 0 1"/>
     </joint>
-    ## rotor arms
-    <link name="rotor_arm${child1}">
-      <inertial>
-        <origin xyz="0.0486 0 0.0161" rpy="0 0 0"/>
-        <mass value="0.088"/>
-        <inertia
-            ixx="0.000001" ixy="0.0" ixz="0.0"
-            iyy="0.0001" iyz="0.0"
-            izz="0.0001"/>
-      </inertial>
-      <visual>
-        <origin xyz="0 0 0" rpy="0 0 0"/>
-        <geometry>
-          <mesh filename="package://gimbalrotor/urdf/quad/mesh/rotor_arm.dae"/>
-        </geometry>
-      </visual>
-      <collision>
-        <origin xyz="0 0 0" rpy="0 0 0"/>
-        <geometry>
-          <box size="0.131 0.0325 0.065"/>
-        </geometry>
-      </collision>
-    </link>
-    <joint name="base_arm_joint${child1}" type="fixed">
-      <parent link="base_link"/>
-      <child link="rotor_arm${child1}"/>
-      <origin rpy="0 0 ${pi/4}" xyz="0.051 0.051 0.0"/>
-      <axis xyz="0 0 1"/>
-    </joint>
-    <link name="rotor_arm${child2}">
-      <inertial>
-        <origin xyz="0.0486 0 0.0161" rpy="0 0 0"/>
-        <mass value="0.088"/>
-        <inertia
-            ixx="0.000001" ixy="0.0" ixz="0.0"
-            iyy="0.0001" iyz="0.0"
-            izz="0.0001"/>
-      </inertial>
-      <visual>
-        <origin xyz="0 0 0" rpy="0 0 0"/>
-        <geometry>
-          <mesh filename="package://gimbalrotor/urdf/quad/mesh/rotor_arm.dae"/>
-        </geometry>
-      </visual>
-      <collision>
-        <origin xyz="0 0 0" rpy="0 0 0"/>
-        <geometry>
-          <box size="0.131 0.0325 0.065"/>
-        </geometry>p
-      </collision>
-    </link>
-    <joint name="base_arm_joint${child2}" type="fixed">
-      <parent link="base_link"/>
-      <child link="rotor_arm${child2}"/>
-      <origin rpy="0 0 ${pi*3.0/4.0}" xyz="-0.051 0.051 0.0"/>
-      <axis xyz="0 0 1"/>
-    </joint>
-    <link name="rotor_arm${child3}">
-      <inertial>
-        <origin xyz="0.0486 0 0.0161" rpy="0 0 0"/>
-        <mass value="0.088"/>
-        <inertia
-            ixx="0.000001" ixy="0.0" ixz="0.0"
-            iyy="0.0001" iyz="0.0"
-            izz="0.0001"/>
-      </inertial>
-      <visual>
-        <origin xyz="0 0 0" rpy="0 0 0"/>
-        <geometry>
-          <mesh filename="package://gimbalrotor/urdf/quad/mesh/rotor_arm.dae"/>
-        </geometry>
-      </visual>
-      <collision>
-        <origin xyz="0 0 0" rpy="0 0 0"/>
-        <geometry>
-          <box size="0.131 0.0325 0.065"/>
-        </geometry>
-      </collision>
-    </link>
-    <joint name="base_arm_joint${child3}" type="fixed">
-      <parent link="base_link"/>
-      <child link="rotor_arm${child3}"/>
-      <origin rpy="0 0 ${pi*5.0/4.0}" xyz="-0.051 -0.051 0.0"/>
-      <axis xyz="0 0 1"/>
-    </joint>
-    <link name="rotor_arm${child4}">
-      <inertial>
-        <origin xyz="0.0486 0 0.0161" rpy="0 0 0"/>
-        <mass value="0.088"/>
-        <inertia
-            ixx="0.000001" ixy="0.0" ixz="0.0"
-            iyy="0.0001" iyz="0.0"
-            izz="0.0001"/>
-      </inertial>
-      <visual>
-        <origin xyz="0 0 0" rpy="0 0 0"/>
-        <geometry>
-          <mesh filename="package://gimbalrotor/urdf/quad/mesh/rotor_arm.dae"/>
-        </geometry>
-      </visual>
-      <collision>
-        <origin xyz="0 0 0" rpy="0 0 0"/>
-        <geometry>
-          <box size="0.131 0.0325 0.065"/>
-        </geometry>
-      </collision>
-    </link>
-    <joint name="base_arm_joint${child4}" type="fixed">
-      <parent link="base_link"/>
-      <child link="rotor_arm${child4}"/>
-      <origin rpy="0 0 ${-pi/4.0}" xyz="0.051 -0.051 0.0"/>
-      <axis xyz="0 0 1"/>
-    </joint>
+    ## rotor arm macro
+    <xacro:macro name="dummy_rotor_arm" params="id x y z yaw">
+      ## link
+      <link name="rotor_arm${id}">
+        <inertial>
+          <origin xyz="0 0 0" rpy="0 0 0"/>
+          <mass value="0.0001"/>
+          <inertia
+              ixx="0.000001" ixy="0.0" ixz="0.0"
+              iyy="0.0001" iyz="0.0"
+              izz="0.0001"/>
+        </inertial>
+      </link>
+      ## joint
+      <joint name="base_arm_joint${id}" type="fixed">
+        <parent link="base_link"/>
+        <child link="rotor_arm${id}"/>
+        <origin rpy="0 0 ${yaw}" xyz="${x} ${y} ${z}"/>
+        <axis xyz="0 0 1"/>
+      </joint>
+    </xacro:macro>
+    ## dummy rotor arms
+    <xacro:dummy_rotor_arm id = "${child1}" x = "0.12041" y="0.12041" z = "0.0555" yaw = "${pi/4.0}"/>
+    <xacro:dummy_rotor_arm id = "${child2}" x = "-0.12129" y="0.12150" z = "0.0555" yaw = "${pi*3.0/4.0}"/>
+    <xacro:dummy_rotor_arm id = "${child3}" x = "-0.12129" y="-0.12150" z = "0.0555" yaw = "${pi*5.0/4.0}"/>
+    <xacro:dummy_rotor_arm id = "${child4}" x = "0.12129" y="-0.12150" z = "0.0555" yaw = "${-pi/4.0}"/>
+    ## dummy link for the contact point coordinate
+      <link name="contact_point">
+        <inertial>
+          <origin xyz="0 0 0" rpy="0 0 0"/>
+          <mass value="0.0001"/>
+          <inertia
+              ixx="0.000001" ixy="0.0" ixz="0.0"
+              iyy="0.0001" iyz="0.0"
+              izz="0.0001"/>
+        </inertial>
+      </link>
+      <joint name="cp_base_joint" type="fixed">
+        <parent link="base_link"/>
+        <child link="contact_point"/>
+        <origin rpy="0 0 0" xyz="0.26 0 0"/>
+        <axis xyz="0 0 1"/>
+      </joint>
     <xacro:friction self="base_link"/>
   </xacro:macro>
@@ -179,14 +109,14 @@
     <link name="gimbal_link${self}">
       <inertial>
-        <origin xyz="0.018 0.00 0.00438" rpy="0 0 0"/>
-        <mass value="0.1095"/>
-        <inertia
-            ixx="0.00002989" iyy="0.00002848" izz="0.0002698"
-            ixy="0.0000" ixz="-0.0000" iyz="0.00000"/>
+        <origin xyz="0.0223521 0.0 0.00776312" rpy="0 0 0"/>
+        <mass value="0.15944"/>
+        <inertia
+            ixx="0.00007458" iyy="0.00007325" izz="0.00007756"
+            ixy="0.00000001" ixz="0.00000084" iyz="0.00000001"/>
       </inertial>
       <collision>
         <origin xyz="0.0 0 0" rpy="0 0 0"/>
         <geometry>
-          <cylinder radius="0.018" length="0.033"/>
+          <cylinder radius="0.02" length="0.033"/>
         </geometry>
       </collision>
@@ -214,5 +144,5 @@
       <inertial>
         <origin xyz="0 0 0" rpy="0 0 0"/>
-        <mass value="0.00001"/>
+        <mass value="0.005"/>
         <inertia
             ixx="0.001" ixy="0.0" ixz="0.0"
@@ -225,8 +155,8 @@
     #### gimbal joints ####
     <joint name="gimbal${self}" type="revolute">
-      <limit effort="6.6" lower="-2.0" upper="2.0" velocity="3.0"/>
+      <limit effort="6.6" lower="-1.57" upper="1.57" velocity="3.0"/>
       <parent link="rotor_arm${self}"/>
       <child link="gimbal_link${self}"/>
-      <origin rpy="0 0 0" xyz="0.077 0 0.0385"/>
+      <origin rpy="0 0 0" xyz="0 0 0"/>
       <axis xyz="1 0 0"/>
       <dynamics damping="0.8" friction="0.0"/>

Commit message: [Beetle_hyper][urdf]change fc pos in Z axis

File: robots/gimbalrotor/urdf/quad/gimbalrotor.urdf.xacro (robot description, xacro)
@@ -56,5 +56,5 @@
       <child link="fc"/>
       <parent link="base_link"/>
-      <origin rpy="0 0 0" xyz="0 0 0"/>
+      <origin rpy="0 0 0" xyz="0 0 0.06747"/>
       <axis xyz="0 0 1"/>
     </joint>
