Commit message: [Beetle][valve]change the valve's urdf into a correct version

File: robots/beetle/urdf/valve.urdf (robot description, URDF)
Before this commit: robot valve, 1 links, 5 joints
Links:
- link handle: geometry visual mesh filename=package://beetle/urdf/mesh/beetle_valve.STL scale=0.001 0.001 0.001
