Commit message: [Beetle_hyper][simulation] workaround on modify the simulation

File: robots/beetle/urdf/valve.urdf (robot description, URDF)
Before this commit: robot valve, 1 links, 5 joints
Links:
- added link world
Joints:
- added joint support_world_joint: type fixed, parent world, child main_pipe, origin xyz=0 0 0 rpy=0 0 0
