Commit message: [Model][urdf] Refacted beetle's urdf file into beetle_hyper's version

File: robots/beetle/urdf/beetle.urdf.xacro (robot description, xacro)
@@ -23,9 +23,9 @@
     <link name="base_link">
       <inertial>
-        <origin xyz="0.0071144 0.0004661 0.1372857" rpy="0 0 0"/>
-        <mass value="2.7703823"/>
-        <inertia
-            ixx="0.0527268" iyy="0.0895178" izz="0.1192811"
-            ixy="-0.0001722" ixz="0.0008599" iyz="0.0000395"/>
+        <origin xyz="0.0257171 0.0007358  0.0813823" rpy="0 0 0"/>
+        <mass value="2.8200834"/>
+        <inertia
+            ixx="0.0679394" iyy="0.1142367" izz=" 0.1213159"
+            ixy="-0.0001621" ixz="0.00612466" iyz="0.0000964"/>
       </inertial>
       <visual>

Commit message: [Beetle_fang][urdf]add end_effctor_fang in gazebo

File: robots/beetle/urdf/beetle.urdf.xacro (robot description, xacro)
@@ -59,56 +59,30 @@
       <axis xyz="0 0 1"/>
     </joint>
-<!-- adding a manipulation link -->
-     <link name="manipulator_link_1">
-      <inertial>
-        <origin xyz="-0.18 0.19 -0.02" rpy="0 0 0"/>
-        <mass value="0.06"/>
-        <inertia
-            ixx="0.0001" iyy="0.0001" izz="0.0001"
-            ixy="0" ixz="0" iyz="0"/>
+<!-- add link for Beetle_fang -->
+     <link name="beetle_fang_link">
+      <inertial>
+        <origin xyz="0.00659 0 -0.01082" rpy="0 0 0"/>
+        <mass value="0.17123"/>
+        <inertia
+            ixx="3.3231" iyy="0.0666" izz="3.2902"
+            ixy="0" ixz="-0.0133" iyz="0"/>
       </inertial>
       <visual>
-        <origin xyz="-0.18 0.19 -0.02" rpy="0 0 3.141592"/>
-        <geometry>
-          <mesh filename="package://beetle/urdf/mesh/manipulator_v1.1.2.dae"/>
+        <origin xyz="0 0 0" rpy="0 0 0"/>
+        <geometry>
+          <mesh filename="package://beetle/urdf/mesh/end_effector_fang.dae"/>
         </geometry>
       </visual>
       <collision>
-        <origin xyz="0.18 0.026 0.019" rpy="0 0 0"/>
-        <geometry>
-          <box size="0.016 0.016 0.5"/>
+        <origin xyz="0 0 0" rpy="0 0 0"/>
+        <geometry>
+          <box size="0.519 0.08411 0.04412"/>
         </geometry>
       </collision>
     </link>
-    <joint name="manipulator_joint_1" type="fixed">
+    <joint name="beetle_fang_joint" type="fixed">
       <parent link="base_link"/>
-      <child link="manipulator_link_1"/>
-      <origin xyz="-0.18 0.19 -0.02" rpy="0 0 0"/>
-    </joint>
-     <link name="manipulator_link_2">
-      <inertial>
-        <origin xyz="-0.18 -0.031 -0.02" rpy="0 0 0"/>
-        <mass value="0.06"/>
-        <inertia
-            ixx="0.0001" iyy="0.0001" izz="0.0001"
-            ixy="0" ixz="0" iyz="0"/>
-      </inertial>
-      <visual>
-        <origin xyz="-0.18 -0.031 -0.02" rpy="0 0 3.141592"/>
-        <geometry>
-          <mesh filename="package://beetle/urdf/mesh/manipulator_v1.1.2.dae"/>
-        </geometry>
-      </visual>
-      <collision>
-        <origin xyz="0.18 -0.196 0.019" rpy="0 0 0"/>
-        <geometry>
-          <box size="0.016 0.016 0.5"/>
-        </geometry>
-      </collision>
-    </link>
-    <joint name="manipulator_joint_2" type="fixed">
-      <parent link="base_link"/>
-      <child link="manipulator_link_2"/>
-      <origin xyz="-0.18 -0.031 -0.02" rpy="0 0 0"/>
+      <child link="beetle_fang_link"/>
+      <origin xyz="0.244 0 0.007" rpy="0 0 0"/>
     </joint>
     ## rotor arm macro
@@ -205,14 +179,4 @@
     </link>
     <xacro:damping_factor link="thrust${self}"/>
-## manipulation link (virtual)
-    <!-- <link name="manipulator_link_1_${self}">
-      <inertial>
-        <origin xyz="0 0 0" rpy="0 0 0"/>
-        <mass value="0.06"/>
-        <inertia
-            ixx="0.000001" iyy="0.000001" izz="0.000001"
-            ixy="0" ixz="0" iyz="0"/>
-      </inertial>
-    </link> -->
     #### joints ####
     #### gimbal joints ####
@@ -250,10 +214,4 @@
       <axis xyz="0 0 ${rotor_direction}"/>
     </joint>
-    #### manipulator joint (virtual) ####
-    <!-- <joint name="manipulator_joint_1_${self}" type="fixed">
-      <parent link="base_link"/>
-      <child link="manipulator_link_1"/>
-      <origin xyz="0.0071144 0.22 0.290" rpy="0 0 0"/>
-    </joint> -->
     <transmission name="rotor_tran${self}">
       <type>transmission_interface/SimpleTransmission</type>

Commit message: [Beetle_fang]adjust empty.world and add fang in urdf

File: robots/beetle/urdf/beetle.urdf.xacro (robot description, xacro)
@@ -35,8 +35,27 @@
         </geometry>
       </visual>
-      <collision>
-        <origin xyz="0 0 0.1205" rpy="0 0 0"/>
-        <geometry>
-          <box size="0.52 0.52 0.241"/>
+      <!-- decompse the collison part for manipulator -->
+      <collision>
+        <origin xyz="-0.042 0 0.1205" rpy="0 0 0"/>
+        <geometry>
+          <box size="0.436 0.52 0.241"/>
+        </geometry>
+      </collision>
+      <collision>
+        <origin xyz="0.218 0 0.14256" rpy="0 0 0"/>
+        <geometry>
+          <box size="0.084 0.52 0.19688"/>
+        </geometry>
+      </collision>
+      <collision>
+        <origin xyz="0.218 0.24 0.02206" rpy="0 0 0"/>
+        <geometry>
+          <box size="0.084 0.040 0.04412"/>
+        </geometry>
+      </collision>
+      <collision>
+        <origin xyz="0.218 -0.24 0.02206" rpy="0 0 0"/>
+        <geometry>
+          <box size="0.084 0.040 0.04412"/>
         </geometry>
       </collision>
@@ -75,7 +94,13 @@
       </visual>
       <collision>
-        <origin xyz="0 0 0" rpy="0 0 0"/>
-        <geometry>
-          <box size="0.519 0.08411 0.04412"/>
+        <origin xyz="0.01 0.06255 -0.0522683" rpy="0 0 0"/>
+        <geometry>
+          <box size="0.012 0.012 0.04412"/>
+        </geometry>
+      </collision>
+      <collision>
+        <origin xyz="0.01 -0.06255 -0.0522683" rpy="0 0 0"/>
+        <geometry>
+          <box size="0.012 0.012 0.04412"/>
         </geometry>
       </collision>
@@ -84,5 +109,5 @@
       <parent link="base_link"/>
       <child link="beetle_fang_link"/>
-      <origin xyz="0.244 0 0.007" rpy="0 0 0"/>
+      <origin xyz="0.244 0 0.0743823" rpy="0 0 0"/>
     </joint>
     ## rotor arm macro

Commit message: [Beetle_fang][urdf]refacted the urdf to fit for the real pos of endeffctor

File: robots/beetle/urdf/beetle.urdf.xacro (robot description, xacro)
@@ -94,5 +94,5 @@
       </visual>
       <collision>
-        <origin xyz="0.01 0.06255 -0.0522683" rpy="0 0 0"/>
+        <origin xyz="0.00772 0.08438 -0.0522683" rpy="0 0 0"/>
         <geometry>
           <box size="0.012 0.012 0.04412"/>
@@ -100,5 +100,5 @@
       </collision>
       <collision>
-        <origin xyz="0.01 -0.06255 -0.0522683" rpy="0 0 0"/>
+        <origin xyz="0.00772 -0.08438 -0.0522683" rpy="0 0 0"/>
         <geometry>
           <box size="0.012 0.012 0.04412"/>

Commit message: [Beetle_fang]fix the error while opening gazebo

File: robots/beetle/urdf/beetle.urdf.xacro (robot description, xacro)
@@ -96,5 +96,5 @@
         <origin xyz="0.00772 0.08438 -0.0522683" rpy="0 0 0"/>
         <geometry>
-          <box size="0.012 0.012 0.04412"/>
+          <cylinder radius="0.006" length="0.04412"/>
         </geometry>
       </collision>
@@ -102,5 +102,5 @@
         <origin xyz="0.00772 -0.08438 -0.0522683" rpy="0 0 0"/>
         <geometry>
-          <box size="0.012 0.012 0.04412"/>
+          <cylinder radius="0.006" length="0.04412"/>
         </geometry>
       </collision>

Commit message: [Beetle_fang][valve rotation]update the trajectory.py

File: robots/beetle/urdf/beetle.urdf.xacro (robot description, xacro)
@@ -94,5 +94,5 @@
       </visual>
       <collision>
-        <origin xyz="0.00772 0.08438 -0.0522683" rpy="0 0 0"/>
+        <origin xyz="0.0072 0.08438 -0.0522683" rpy="0 0 0"/>
         <geometry>
           <cylinder radius="0.006" length="0.04412"/>
@@ -109,5 +109,5 @@
       <parent link="base_link"/>
       <child link="beetle_fang_link"/>
-      <origin xyz="0.244 0 0.0743823" rpy="0 0 0"/>
+      <origin xyz="0.246 0 0.0743823" rpy="0 0 0"/>
     </joint>
     ## rotor arm macro

File: robots/beetle/urdf/valve.urdf (robot description, URDF)
Before this commit: robot valve, 2 links, 6 joints
Links:
- removed link i_beam
Joints:
- removed joint valve_to_i_beam_joint

Commit message: [Beetle_fang]changing urdf into Beetle_fang's version

File: robots/beetle/urdf/beetle.urdf.xacro (robot description, xacro)
@@ -35,8 +35,27 @@
         </geometry>
       </visual>
-      <collision>
-        <origin xyz="0 0 0.1205" rpy="0 0 0"/>
-        <geometry>
-          <box size="0.52 0.52 0.241"/>
+      <!-- decompse the collison part for manipulator -->
+      <collision>
+        <origin xyz="-0.042 0 0.1205" rpy="0 0 0"/>
+        <geometry>
+          <box size="0.436 0.52 0.241"/>
+        </geometry>
+      </collision>
+      <collision>
+        <origin xyz="0.218 0 0.14256" rpy="0 0 0"/>
+        <geometry>
+          <box size="0.084 0.52 0.19688"/>
+        </geometry>
+      </collision>
+      <collision>
+        <origin xyz="0.218 0.24 0.02206" rpy="0 0 0"/>
+        <geometry>
+          <box size="0.084 0.040 0.04412"/>
+        </geometry>
+      </collision>
+      <collision>
+        <origin xyz="0.218 -0.24 0.02206" rpy="0 0 0"/>
+        <geometry>
+          <box size="0.084 0.040 0.04412"/>
         </geometry>
       </collision>
@@ -58,4 +77,37 @@
       <origin rpy="0 0 0" xyz="0 0 0.12947"/>
       <axis xyz="0 0 1"/>
+    </joint>
+<!-- add link for Beetle_fang -->
+     <link name="beetle_fang_link">
+      <inertial>
+        <origin xyz="0.00659 0 -0.01082" rpy="0 0 0"/>
+        <mass value="0.17123"/>
+        <inertia
+            ixx="3.3231" iyy="0.0666" izz="3.2902"
+            ixy="0" ixz="-0.0133" iyz="0"/>
+      </inertial>
+      <visual>
+        <origin xyz="0 0 0" rpy="0 0 0"/>
+        <geometry>
+          <mesh filename="package://beetle/urdf/mesh/end_effector_fang.dae"/>
+        </geometry>
+      </visual>
+      <collision>
+        <origin xyz="0.0072 0.08438 -0.0522683" rpy="0 0 0"/>
+        <geometry>
+          <cylinder radius="0.006" length="0.04412"/>
+        </geometry>
+      </collision>
+      <collision>
+        <origin xyz="0.00772 -0.08438 -0.0522683" rpy="0 0 0"/>
+        <geometry>
+          <cylinder radius="0.006" length="0.04412"/>
+        </geometry>
+      </collision>
+    </link>
+    <joint name="beetle_fang_joint" type="fixed">
+      <parent link="base_link"/>
+      <child link="beetle_fang_link"/>
+      <origin xyz="0.246 0 0.0743823" rpy="0 0 0"/>
     </joint>
     ## rotor arm macro

Commit message: [Beetle][urdf]adjust the pos of cog in x axis to fix error in pitch while taking off

File: robots/beetle/urdf/beetle.urdf.xacro (robot description, xacro)
@@ -23,5 +23,6 @@
     <link name="base_link">
       <inertial>
-        <origin xyz="0.0071144 0.0004661 0.1372857" rpy="0 0 0"/>
+        <!-- <origin xyz="0.0071144 0.0004661 0.1372857" rpy="0 0 0"/> -->
+        <origin xyz="-0.009 0.0004661 0.1372857" rpy="0 0 0"/>
         <mass value="2.7703823"/>
         <inertia

Commit message: [Beetle][urdf]update urdf of beetle

File: robots/beetle/urdf/beetle.urdf.xacro (robot description, xacro)
@@ -24,5 +24,5 @@
       <inertial>
         <!-- <origin xyz="0.0071144 0.0004661 0.1372857" rpy="0 0 0"/> -->
-        <origin xyz="-0.009 0.0004661 0.1372857" rpy="0 0 0"/>
+        <origin xyz="-0.013 0.0004661 0.1372857" rpy="0 0 0"/>
         <mass value="2.7703823"/>
         <inertia

Commit message: [Beetle][urdf]Update cog pos of baselink

File: robots/beetle/urdf/beetle.urdf.xacro (robot description, xacro)
@@ -24,5 +24,5 @@
       <inertial>
         <!-- <origin xyz="0.0071144 0.0004661 0.1372857" rpy="0 0 0"/> -->
-        <origin xyz="-0.013 0.0004661 0.1372857" rpy="0 0 0"/>
+        <origin xyz="-0.016 0.0004661 0.1372857" rpy="0 0 0"/>
         <mass value="2.7703823"/>
         <inertia

Commit message: [Beetle_hyper][urdf] change beetle's urdf into beetle_hyper's version

File: robots/beetle/urdf/beetle.urdf.xacro (robot description, xacro)
@@ -23,9 +23,9 @@
     <link name="base_link">
       <inertial>
-        <origin xyz="0.0071144 0.0004661 0.1372857" rpy="0 0 0"/>
-        <mass value="2.7703823"/>
-        <inertia
-            ixx="0.0527268" iyy="0.0895178" izz="0.1192811"
-            ixy="-0.0001722" ixz="0.0008599" iyz="0.0000395"/>
+        <origin xyz="0.0257171 0.0007358  0.0813823" rpy="0 0 0"/>
+        <mass value="2.8200834"/>
+        <inertia
+            ixx="0.0679394" iyy="0.1142367" izz="0.1213159"
+            ixy="-0.0001621" ixz="0.00612466" iyz="0.0000964"/>
       </inertial>
       <visual>

File: robots/beetle/urdf/beetle_fang.urdf.xacro (robot description, xacro)
@@ -23,9 +23,9 @@
     <link name="base_link">
       <inertial>
-        <origin xyz="0.0071144 0.0004661 0.1372857" rpy="0 0 0"/>
-        <mass value="2.7703823"/>
-        <inertia
-            ixx="0.0527268" iyy="0.0895178" izz="0.1192811"
-            ixy="-0.0001722" ixz="0.0008599" iyz="0.0000395"/>
+        <origin xyz="0.0257171 0.0007358  0.0813823" rpy="0 0 0"/>
+        <mass value="2.8200834"/>
+        <inertia
+            ixx="0.0679394" iyy="0.1142367" izz="0.1213159"
+            ixy="-0.0001621" ixz="0.00612466" iyz="0.0000964"/>
       </inertial>
       <visual>

Commit message: [Beetle_hyper][urdf] change inertial matrix into correct one

File: robots/beetle/urdf/beetle.urdf.xacro (robot description, xacro)
@@ -23,12 +23,11 @@
     <link name="base_link">
       <inertial>
-        <origin xyz="0.0257171 0.0007358  0.0813823" rpy="0 0 0"/>
-        <mass value="2.8200834"/>
+        <origin xyz="0.0064914 0.0007538  0.0774673" rpy="0 0 0"/>
+        <mass value="2.7584217"/>
         <inertia
-            ixx="0.0679394" iyy="0.1142367" izz="0.1213159"
-            ixy="-0.0001621" ixz="0.00612466" iyz="0.0000964"/>
+            ixx="0.0521449" iyy="0.0872700" izz="0.1157478"
+            ixy="-0.0001753" ixz="0.0004696" iyz="-0.0000646"/>
       </inertial>
       <visual>
-        <origin xyz="0 0 0" rpy="0 0 3.141592"/>
         <geometry>
           <mesh filename="package://beetle/urdf/mesh/base_link_hyper.dae"/>

File: robots/beetle/urdf/beetle_fang.urdf.xacro (robot description, xacro)
@@ -23,9 +23,9 @@
     <link name="base_link">
       <inertial>
-        <origin xyz="0.0257171 0.0007358  0.0813823" rpy="0 0 0"/>
-        <mass value="2.8200834"/>
-        <inertia
-            ixx="0.0679394" iyy="0.1142367" izz="0.1213159"
-            ixy="-0.0001621" ixz="0.00612466" iyz="0.0000964"/>
+        <origin xyz="0.0064914 0.0007538  0.0774673" rpy="0 0 0"/>
+        <mass value="2.7584217"/>
+        <inertia
+            ixx="0.0521449" iyy="0.0872700" izz="0.1157478"
+            ixy="-0.0001753" ixz="0.0004696" iyz="-0.0000646"/>
       </inertial>
       <visual>

Commit message: [Beetle_hyper][urdf] fix the bug in urdf for visualize the beetle in gazebo

File: robots/beetle/urdf/beetle.urdf.xacro (robot description, xacro)
@@ -30,4 +30,5 @@
       </inertial>
       <visual>
+        <origin xyz="0 0 0" rpy="0 0 3.141592"/>
         <geometry>
           <mesh filename="package://beetle/urdf/mesh/base_link_hyper.dae"/>
