Commit message: [Beetle_hyper][urdf] modify beetle_hyper's urdf  based on experiment

File: robots/beetle/urdf/beetle.urdf.xacro (robot description, xacro)
@@ -24,5 +24,5 @@
       <inertial>
         <origin xyz="0.0064914 0.0007538  0.0774673" rpy="0 0 0"/>
-        <mass value="2.7584217"/>
+        <mass value="2.8122407"/>
         <inertia
             ixx="0.059467" iyy="0.092209" izz="0.128586"

File: robots/beetle/urdf/beetle_fang.urdf.xacro (robot description, xacro)
@@ -24,7 +24,7 @@
       <inertial>
         <origin xyz="0.0064914 0.0007538  0.0774673" rpy="0 0 0"/>
-        <mass value="2.7584217"/>
-        <inertia
-            ixx="0.0521449" iyy="0.0872700" izz="0.1157478"
+        <mass value="2.8122407"/>
+        <inertia
+            ixx="0.059467" iyy="0.092209" izz="0.128586"
             ixy="-0.0001753" ixz="0.0004696" iyz="-0.0000646"/>
       </inertial>

Commit message: [Beetle_hyper][urdf] adjust cog pos based on hovering calibration

File: robots/beetle/urdf/beetle.urdf.xacro (robot description, xacro)
@@ -23,5 +23,5 @@
     <link name="base_link">
       <inertial>
-        <origin xyz="0.0064914 0.0007538  0.0774673" rpy="0 0 0"/>
+        <origin xyz="0.0254914 0.0027538  0.0774673" rpy="0 0 0"/>
         <mass value="2.8122407"/>
         <inertia

File: robots/beetle/urdf/beetle_fang.urdf.xacro (robot description, xacro)
@@ -23,5 +23,5 @@
     <link name="base_link">
       <inertial>
-        <origin xyz="0.0064914 0.0007538  0.0774673" rpy="0 0 0"/>
+        <origin xyz="0.0254914 0.0027538  0.0774673" rpy="0 0 0"/>
         <mass value="2.8122407"/>
         <inertia

Commit message: [Beetle_hyper][urdf] adjust cog

File: robots/beetle/urdf/beetle.urdf.xacro (robot description, xacro)
@@ -23,5 +23,5 @@
     <link name="base_link">
       <inertial>
-        <origin xyz="0.0254914 0.0027538  0.0774673" rpy="0 0 0"/>
+        <origin xyz="0.0124914 0.0027538  0.0774673" rpy="0 0 0"/>
         <mass value="2.8122407"/>
         <inertia

File: robots/beetle/urdf/beetle_fang.urdf.xacro (robot description, xacro)
@@ -23,5 +23,5 @@
     <link name="base_link">
       <inertial>
-        <origin xyz="0.0254914 0.0027538  0.0774673" rpy="0 0 0"/>
+        <origin xyz="0.0124914 0.0027538  0.0774673" rpy="0 0 0"/>
         <mass value="2.8122407"/>
         <inertia

Commit message: [Beetle_hyper][urdf] modify cog pos

File: robots/beetle/urdf/beetle.urdf.xacro (robot description, xacro)
@@ -23,5 +23,5 @@
     <link name="base_link">
       <inertial>
-        <origin xyz="0.0124914 0.0027538  0.0774673" rpy="0 0 0"/>
+        <origin xyz="0.0154914 0.0027538  0.0774673" rpy="0 0 0"/>
         <mass value="2.8122407"/>
         <inertia

File: robots/beetle/urdf/beetle_fang.urdf.xacro (robot description, xacro)
@@ -23,5 +23,5 @@
     <link name="base_link">
       <inertial>
-        <origin xyz="0.0124914 0.0027538  0.0774673" rpy="0 0 0"/>
+        <origin xyz="0.0154914 0.0027538  0.0774673" rpy="0 0 0"/>
         <mass value="2.8122407"/>
         <inertia

Commit message: [Beetle_hyper][urdf] cog adjust

File: robots/beetle/urdf/beetle.urdf.xacro (robot description, xacro)
@@ -23,5 +23,5 @@
     <link name="base_link">
       <inertial>
-        <origin xyz="0.0154914 0.0027538  0.0774673" rpy="0 0 0"/>
+        <origin xyz="0.0174914 0.0027538  0.0774673" rpy="0 0 0"/>
         <mass value="2.8122407"/>
         <inertia

File: robots/beetle/urdf/beetle_fang.urdf.xacro (robot description, xacro)
@@ -23,5 +23,5 @@
     <link name="base_link">
       <inertial>
-        <origin xyz="0.0154914 0.0027538  0.0774673" rpy="0 0 0"/>
+        <origin xyz="0.0174914 0.0027538  0.0774673" rpy="0 0 0"/>
         <mass value="2.8122407"/>
         <inertia
