Commit message: [Beetle][Wrench-type valve opening]Support spawning n modules in gazebo with different urdf

File: robots/beetle/urdf/beetle_fang.urdf.xacro (robot description, xacro)
@@ -35,8 +35,27 @@
         </geometry>
       </visual>
-      <collision>
-        <origin xyz="0 0 0.1205" rpy="0 0 0"/>
-        <geometry>
-          <box size="0.52 0.52 0.241"/>
+      <!-- decompse the collison part for manipulator -->
+      <collision>
+        <origin xyz="-0.042 0 0.1205" rpy="0 0 0"/>
+        <geometry>
+          <box size="0.436 0.52 0.241"/>
+        </geometry>
+      </collision>
+      <collision>
+        <origin xyz="0.218 0 0.14256" rpy="0 0 0"/>
+        <geometry>
+          <box size="0.084 0.52 0.19688"/>
+        </geometry>
+      </collision>
+      <collision>
+        <origin xyz="0.218 0.24 0.02206" rpy="0 0 0"/>
+        <geometry>
+          <box size="0.084 0.040 0.04412"/>
+        </geometry>
+      </collision>
+      <collision>
+        <origin xyz="0.218 -0.24 0.02206" rpy="0 0 0"/>
+        <geometry>
+          <box size="0.084 0.040 0.04412"/>
         </geometry>
       </collision>
@@ -58,4 +77,37 @@
       <origin rpy="0 0 0" xyz="0 0 0.12947"/>
       <axis xyz="0 0 1"/>
+    </joint>
+<!-- add link for Beetle_fang -->
+     <link name="beetle_fang_link">
+      <inertial>
+        <origin xyz="0.00659 0 -0.01082" rpy="0 0 0"/>
+        <mass value="0.17123"/>
+        <inertia
+            ixx="0.0033" iyy="0.0" izz="0.00329"
+            ixy="0.0" ixz="-0.000013" iyz="0.0"/>
+      </inertial>
+      <visual>
+        <origin xyz="0 0 0" rpy="0 0 0"/>
+        <geometry>
+          <mesh filename="package://beetle/urdf/mesh/end_effector_fang.dae"/>
+        </geometry>
+      </visual>
+      <collision>
+        <origin xyz="0.0072 0.08438 -0.0522683" rpy="0 0 0"/>
+        <geometry>
+          <cylinder radius="0.006" length="0.04412"/>
+        </geometry>
+      </collision>
+      <collision>
+        <origin xyz="0.00772 -0.08438 -0.0522683" rpy="0 0 0"/>
+        <geometry>
+          <cylinder radius="0.006" length="0.04412"/>
+        </geometry>
+      </collision>
+    </link>
+    <joint name="beetle_fang_joint" type="fixed">
+      <parent link="base_link"/>
+      <child link="beetle_fang_link"/>
+      <origin xyz="0.246 0 0.0743823" rpy="0 0 0"/>
     </joint>
     ## rotor arm macro

Commit message: [Beetle][valve rotation] Change the distance bewteen two fang from 186mm to 150mm to support better insertation

File: robots/beetle/urdf/beetle_fang.urdf.xacro (robot description, xacro)
@@ -84,15 +84,15 @@
         <mass value="0.17123"/>
         <inertia
-            ixx="0.0033" iyy="0.0" izz="0.00329"
-            ixy="0.0" ixz="-0.000013" iyz="0.0"/>
+            ixx="0.00327" iyy="0.00007" izz="0.00324"
+            ixy="0.00000" ixz="-0.00001" iyz="0.00001"/>
       </inertial>
       <visual>
         <origin xyz="0 0 0" rpy="0 0 0"/>
         <geometry>
-          <mesh filename="package://beetle/urdf/mesh/end_effector_fang.dae"/>
+          <mesh filename="package://beetle/urdf/mesh/end_effector_fang_150 .dae"/>
         </geometry>
       </visual>
       <collision>
-        <origin xyz="0.0072 0.08438 -0.0522683" rpy="0 0 0"/>
+        <origin xyz="0.0072 0.075 -0.0522683" rpy="0 0 0"/>
         <geometry>
           <cylinder radius="0.006" length="0.04412"/>
@@ -100,5 +100,5 @@
       </collision>
       <collision>
-        <origin xyz="0.00772 -0.08438 -0.0522683" rpy="0 0 0"/>
+        <origin xyz="0.00772 -0.075 -0.0522683" rpy="0 0 0"/>
         <geometry>
           <cylinder radius="0.006" length="0.04412"/>

Commit message: [Beetle_fang]Changing the distance between fang into 150mm to support better insertation

File: robots/beetle/urdf/beetle_fang.urdf.xacro (robot description, xacro)
@@ -84,15 +84,15 @@
         <mass value="0.17123"/>
         <inertia
-            ixx="0.0033" iyy="0.0" izz="0.00329"
-            ixy="0.0" ixz="-0.000013" iyz="0.0"/>
+            ixx="0.00327" iyy="0.00007" izz="0.00324"
+            ixy="0.00000" ixz="-0.00001" iyz="0.00001"/>
       </inertial>
       <visual>
         <origin xyz="0 0 0" rpy="0 0 0"/>
         <geometry>
-          <mesh filename="package://beetle/urdf/mesh/end_effector_fang.dae"/>
+          <mesh filename="package://beetle/urdf/mesh/end_effector_fang_150.dae"/>
         </geometry>
       </visual>
       <collision>
-        <origin xyz="0.0072 0.08438 -0.0522683" rpy="0 0 0"/>
+        <origin xyz="0.0072 0.075 -0.0522683" rpy="0 0 0"/>
         <geometry>
           <cylinder radius="0.006" length="0.04412"/>
@@ -100,5 +100,5 @@
       </collision>
       <collision>
-        <origin xyz="0.00772 -0.08438 -0.0522683" rpy="0 0 0"/>
+        <origin xyz="0.00772 -0.075 -0.0522683" rpy="0 0 0"/>
         <geometry>
           <cylinder radius="0.006" length="0.04412"/>

Commit message: [Beetle][valve rotation demo] fix geometry bugs in calculation

File: robots/beetle/urdf/beetle_fang.urdf.xacro (robot description, xacro)
@@ -90,5 +90,5 @@
         <origin xyz="0 0 0" rpy="0 0 0"/>
         <geometry>
-          <mesh filename="package://beetle/urdf/mesh/end_effector_fang_150 .dae"/>
+          <mesh filename="package://beetle/urdf/mesh/end_effector_fang_150.dae"/>
         </geometry>
       </visual>

Commit message: [Beetle][valve rotation demo] First robust version of valve opertation task by single drone, leaving-valve motion still need to be modified

File: robots/beetle/urdf/beetle_fang.urdf.xacro (robot description, xacro)
@@ -37,25 +37,25 @@
       <!-- decompse the collison part for manipulator -->
       <collision>
-        <origin xyz="-0.042 0 0.1205" rpy="0 0 0"/>
-        <geometry>
-          <box size="0.436 0.52 0.241"/>
-        </geometry>
-      </collision>
-      <collision>
-        <origin xyz="0.218 0 0.14256" rpy="0 0 0"/>
-        <geometry>
-          <box size="0.084 0.52 0.19688"/>
-        </geometry>
-      </collision>
-      <collision>
-        <origin xyz="0.218 0.24 0.02206" rpy="0 0 0"/>
-        <geometry>
-          <box size="0.084 0.040 0.04412"/>
-        </geometry>
-      </collision>
-      <collision>
-        <origin xyz="0.218 -0.24 0.02206" rpy="0 0 0"/>
-        <geometry>
-          <box size="0.084 0.040 0.04412"/>
+        <origin xyz="-0.09 0 0.1205" rpy="0 0 0"/>
+        <geometry>
+          <box size="0.34 0.52 0.241"/>
+        </geometry>
+      </collision>
+      <collision>
+        <origin xyz="0.17 0 0.14256" rpy="0 0 0"/>
+        <geometry>
+          <box size="0.18 0.52 0.19688"/>
+        </geometry>
+      </collision>
+      <collision>
+        <origin xyz="0.17 0.24 0.02206" rpy="0 0 0"/>
+        <geometry>
+          <box size="0.18 0.040 0.04412"/>
+        </geometry>
+      </collision>
+      <collision>
+        <origin xyz="0.17 -0.24 0.02206" rpy="0 0 0"/>
+        <geometry>
+          <box size="0.18 0.040 0.04412"/>
         </geometry>
       </collision>

Commit message: [Beetle][urdf]update urdf of beetle_fang

File: robots/beetle/urdf/beetle_fang.urdf.xacro (robot description, xacro)
@@ -23,5 +23,5 @@
     <link name="base_link">
       <inertial>
-        <origin xyz="0.0071144 0.0004661 0.1372857" rpy="0 0 0"/>
+        <origin xyz="-0.0040 0.0004661 0.1372857" rpy="0 0 0"/>
         <mass value="2.7703823"/>
         <inertia

Commit message: [Beetle_hyper][aerial towing] first demo of aerial_towing by beetle_hyper

File: robots/beetle/urdf/beetle_fang.urdf.xacro (robot description, xacro)
@@ -111,4 +111,13 @@
       <origin xyz="0.246 0 0.0113823" rpy="0 0 0"/>
     </joint>
+    <!-- Gazebo碰撞属性 - 高摩擦防止滑动 -->
+    <gazebo reference="beetle_fang_link">
+      <mu1>10.0</mu1>
+      <mu2>10.0</mu2>
+      <kp>1000000.0</kp>
+      <kd>100.0</kd>
+      <minDepth>0.001</minDepth>
+      <maxVel>0.5</maxVel>
+    </gazebo>
     ## rotor arm macro
     <xacro:macro name="dummy_rotor_arm" params="id x y z yaw">

File: robots/beetle/urdf/load.urdf (robot description, URDF)
Before this commit: robot load, 3 links, 2 joints
Links:
- link slide_x: mass 0.001 -> 0.1; geometry visual sphere radius=0.01

Commit message: [Beetle_hyper][manipulation] modified aerial towing part for real-world experiment

File: robots/beetle/urdf/beetle_fang.urdf.xacro (robot description, xacro)
@@ -49,13 +49,13 @@
       </collision>
       <collision>
-        <origin xyz="0.17 0.24 -0.04094" rpy="0 0 0"/>
-        <geometry>
-          <box size="0.18 0.040 0.04412"/>
-        </geometry>
-      </collision>
-      <collision>
-        <origin xyz="0.17 -0.24 -0.04094" rpy="0 0 0"/>
-        <geometry>
-          <box size="0.18 0.040 0.04412"/>
+        <origin xyz="0.245 0.24 -0.04094" rpy="0 0 0"/>
+        <geometry>
+          <box size="0.03 0.040 0.04412"/>
+        </geometry>
+      </collision>
+      <collision>
+        <origin xyz="0.245 -0.24 -0.04094" rpy="0 0 0"/>
+        <geometry>
+          <box size="0.03 0.040 0.04412"/>
         </geometry>
       </collision>

Commit message: [Beetle_hyper][urdf] modified urdf model of Beetle_hyper and load to fit real-world exp

File: robots/beetle/urdf/beetle_fang.urdf.xacro (robot description, xacro)
@@ -103,4 +103,23 @@
         <geometry>
           <cylinder radius="0.006" length="0.04412"/>
+        </geometry>
+      </collision>
+      <!-- ========================================================= -->
+      <!-- Optional hook collision boxes for gripping the frame       -->
+      <!-- Uncomment this block to enable hooks; comment it to disable -->
+      <!-- Hook size: x=40mm, y=20mm, z=5mm                           -->
+      <!-- Bottom face aligned with fang bottom end                   -->
+      <!-- Extends toward negative x direction in body frame          -->
+      <!-- ========================================================= -->
+      <collision>
+        <origin xyz="-0.0188 0.075 -0.0718283" rpy="0 0 0"/>
+        <geometry>
+          <box size="0.04 0.02 0.005"/>
+        </geometry>
+      </collision>
+      <collision>
+        <origin xyz="-0.01828 -0.075 -0.0718283" rpy="0 0 0"/>
+        <geometry>
+          <box size="0.04 0.02 0.005"/>
         </geometry>
       </collision>

File: robots/beetle/urdf/load.urdf (robot description, URDF)
Before this commit: robot load, 3 links, 2 joints
Links:
- link load_box: geometry collision box size=${box_length} ${box_width} ${wall_thickness}; collision box size=${wall_thickness} ${box_width - 2*wall_thickness} ${wall_th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

Commit message: [Beetle_hyper][urdf] modifed urdf to fit the real model

File: robots/beetle/urdf/beetle_fang.urdf.xacro (robot description, xacro)
@@ -51,5 +51,5 @@
         <origin xyz="0.245 0.24 -0.04094" rpy="0 0 0"/>
         <geometry>
-          <box size="0.03 0.040 0.04412"/>
+          <cylinder radius="0.013" length="0.04412"/>
         </geometry>
       </collision>
@@ -57,5 +57,5 @@
         <origin xyz="0.245 -0.24 -0.04094" rpy="0 0 0"/>
         <geometry>
-          <box size="0.03 0.040 0.04412"/>
+          <cylinder radius="0.013" length="0.04412"/>
         </geometry>
       </collision>
@@ -113,13 +113,13 @@
       <!-- ========================================================= -->
       <collision>
-        <origin xyz="-0.0188 0.075 -0.0718283" rpy="0 0 0"/>
-        <geometry>
-          <box size="0.04 0.02 0.005"/>
-        </geometry>
-      </collision>
-      <collision>
-        <origin xyz="-0.01828 -0.075 -0.0718283" rpy="0 0 0"/>
-        <geometry>
-          <box size="0.04 0.02 0.005"/>
+        <origin xyz="-0.0243 0.075 -0.0718283" rpy="0 0 0"/>
+        <geometry>
+          <box size="0.051 0.02 0.005"/>
+        </geometry>
+      </collision>
+      <collision>
+        <origin xyz="-0.02378 -0.075 -0.0718283" rpy="0 0 0"/>
+        <geometry>
+          <box size="0.051 0.02 0.005"/>
         </geometry>
       </collision>
