Commit message: [Beetle_hyper][urdf] modify weight of end-effector according to the ground truth valve

File: robots/beetle/urdf/beetle_fang.urdf.xacro (robot description, xacro)
@@ -82,5 +82,5 @@
       <inertial>
         <origin xyz="0.00659 0 -0.01082" rpy="0 0 0"/>
-        <mass value="0.17123"/>
+        <mass value="0.37"/>
         <inertia
             ixx="0.00327" iyy="0.00007" izz="0.00324"

Commit message: fix(beetle): use windowed stall detection for wall contact
Keep simulation and real-machine wall pushing on the same default
stall-based contact gate, but replace instantaneous velocity gating with
a short-window progress check to avoid false timeouts from pose jitter.

File: robots/beetle/urdf/beetle_fang.urdf.xacro (robot description, xacro)
@@ -82,5 +82,5 @@
       <inertial>
         <origin xyz="0.00659 0 -0.01082" rpy="0 0 0"/>
-        <mass value="0.37"/>
+        <mass value="0.25"/>
         <inertia
             ixx="0.00327" iyy="0.00007" izz="0.00324"

Commit message: [Beetle_hyper][unified] bound QP allocation by dynamic thrust limit

File: robots/beetle/urdf/beetle_fang.urdf.xacro (robot description, xacro)
@@ -82,5 +82,5 @@
       <inertial>
         <origin xyz="0.00659 0 -0.01082" rpy="0 0 0"/>
-        <mass value="0.25"/>
+        <mass value="0.24"/>
         <inertia
             ixx="0.00327" iyy="0.00007" izz="0.00324"
