Commit message: [Beetle][demo] add movable/fixed wall switch for static vs dynamic push in sim
wall.urdf: wall_joint is now conditional on wall_static (default true):
 - true  -> fixed joint to world: anchored wall = static force test (the FT
            sensor at wall_joint still reads the push force);
 - false -> prismatic joint along the push axis (X) with Coulomb friction and
            damping, so a push exceeding wall_slide_friction slides the wall in
            the plane without tipping = dynamic push. FT sensor + /wall/odom are
            kept for both modes.

Plumb wall_static / wall_slide_friction / wall_slide_damping through
wall_pos.launch and wall_pushing_formation.launch. Pair wall_static:=false with
the demo's push_move_distance:=0.5 for the dynamic experiment.

xacro validated for both modes (fixed vs prismatic); launch XML validated.
Default unchanged (fixed wall).

Co-Authored-By: Claude Opus 4.8 <noreply@anthropic.com>

File: robots/beetle/urdf/wall.urdf (robot description, URDF)
Before this commit: robot wall, 2 links, 1 joints
Joints:
- removed joint wall_joint
