Commit message: [Beetle_hyper][demo]: rework static downward valve wrench test
- fix the downward valve and rotate its holder yaw by 45 degrees
- reuse valve-centred arc motion for angular-stall contact detection
- ramp, hold and unload a full 6D application-point wrench at the formation CoG
- remove redundant experiment gates and legacy torque-test helpers
- add tests for stall detection, wrench routing and abnormal cleanup

File: robots/beetle/urdf/valve_downward.urdf (robot description, URDF)
Before this commit: robot valve_downward, 2 links, 6 joints
Joints:
- joint valve_joint: axis 0 0 1 -> (none); type continuous -> fixed
