Commit message: [TRADY]Fix the bug in collision box

File: robots/assemble_quadrotors/urdf/assemble_dual_quadrotors_male_mag.gazebo.xacro (robot description, xacro)
@@ -11,4 +11,8 @@
     <mu1>0.1</mu1>
     <mu2>0.1</mu2>
+    <!-- Using damping factor to stop drifting -->
+    <dampingFactor>0.01</dampingFactor>
+    <kp>1000000.0</kp>
+    <kd>1.0</kd>
   </gazebo>
   <!-- gazebo plugin for docking mech -->

File: robots/assemble_quadrotors/urdf/assemble_dual_quadrotors_male_mag.urdf.xacro (robot description, xacro)
@@ -24,5 +24,6 @@
   <xacro:macro name="damping_factor" params="link">
     <gazebo reference="main_body">
-      <dampingFactor>0.00</dampingFactor>
+      <!-- 增加阻尼来抑制漂移，原值0.00 -->
+      <dampingFactor>0.01</dampingFactor>
     </gazebo>
   </xacro:macro>
@@ -125,5 +126,6 @@
       <origin rpy="0 0 0" xyz="0 0 0"/>
       <geometry>
-        <box size="0.3525 0.26 0.092" />
+        <!--Fix the size of collision box -->
+        <box size="0.3525 0.35 0.19" />
       </geometry>
     </collision>

File: robots/assemble_quadrotors/urdf/robot.urdf.xacro (robot description, xacro)
@@ -117,5 +117,5 @@
       <origin rpy="0 0 0" xyz="0 0 0"/>
       <geometry>
-        <box size="0.26 0.26 0.0575" />
+        <box size="0.26 0.26 0.575" />
       </geometry>
     </collision>
