Commit message: [Beetle][urdf]change the x pos of cog into correct valve to aviod pitch error

File: robots/beetle/robots/beetle.urdf.xacro (robot description, xacro)
@@ -77,47 +77,47 @@
   </link>
   <!-- battery -->
-  <joint name="battery1_joint" type="fixed">
-    <parent link="base_link"/>
-    <child link="battery1"/>
-    <origin xyz="0 0.044 0.055" rpy="0 0 0"/>
-    <axis xyz="1 0 0"/>
-  </joint>
-  <link name="battery1">
-    <inertial>
-      <origin xyz="0 0 -0.017" rpy="0 0 0"/>
-      <mass value="0.41"/>
-      <inertia
-          ixx="0.00060259" ixy="0.0" ixz="0.0"
-          iyy="0.00062827" iyz="0.0"
-          izz="0.00010170"/>
-    </inertial>
-    <visual>
-      <origin rpy="0 0 0" xyz="0 0 -0.017"/>
-      <geometry>
-        <box size="0.13 0.044 0.034"/>
-      </geometry>
-    </visual>
-  </link>
-  <joint name="battery2_joint" type="fixed">
-    <parent link="base_link"/>
-    <child link="battery2"/>
-    <origin xyz="0 -0.044 0.055" rpy="0 0 0"/>
-    <axis xyz="1 0 0"/>
-  </joint>
-  <link name="battery2">
-    <inertial>
-      <origin xyz="0 0 -0.017" rpy="0 0 0"/>
-      <mass value="0.41"/>
-      <inertia
-          ixx="0.00060259" ixy="0.0" ixz="0.0"
-          iyy="0.00062827" iyz="0.0"
-          izz="0.00010170"/>
-    </inertial>
-    <visual>
-      <origin rpy="0 0 0" xyz="0 0 -0.017"/>
-      <geometry>
-        <box size="0.13 0.044 0.034"/>
-      </geometry>
-    </visual>
-  </link>
+  <!-- <joint name="battery1_joint" type="fixed"> -->
+  <!--   <parent link="base_link"/> -->
+  <!--   <child link="battery1"/> -->
+  <!--   <origin xyz="0 0.044 0.055" rpy="0 0 0"/> -->
+  <!--   <axis xyz="1 0 0"/> -->
+  <!-- </joint> -->
+  <!-- <link name="battery1"> -->
+  <!--   <inertial> -->
+  <!--     <origin xyz="0 0 -0.017" rpy="0 0 0"/> -->
+  <!--     <mass value="0.41"/> -->
+  <!--     <inertia -->
+  <!--         ixx="0.00060259" ixy="0.0" ixz="0.0" -->
+  <!--         iyy="0.00062827" iyz="0.0" -->
+  <!--         izz="0.00010170"/> -->
+  <!--   </inertial> -->
+  <!--   <visual> -->
+  <!--     <origin rpy="0 0 0" xyz="0 0 -0.017"/> -->
+  <!--     <geometry> -->
+  <!--       <box size="0.13 0.044 0.034"/> -->
+  <!--     </geometry> -->
+  <!--   </visual> -->
+  <!-- </link> -->
+  <!-- <joint name="battery2_joint" type="fixed"> -->
+  <!--   <parent link="base_link"/> -->
+  <!--   <child link="battery2"/> -->
+  <!--   <origin xyz="0 -0.044 0.055" rpy="0 0 0"/> -->
+  <!--   <axis xyz="1 0 0"/> -->
+  <!-- </joint> -->
+  <!-- <link name="battery2"> -->
+  <!--   <inertial> -->
+  <!--     <origin xyz="0 0 -0.017" rpy="0 0 0"/> -->
+  <!--     <mass value="0.41"/> -->
+  <!--     <inertia -->
+  <!--         ixx="0.00060259" ixy="0.0" ixz="0.0" -->
+  <!--         iyy="0.00062827" iyz="0.0" -->
+  <!--         izz="0.00010170"/> -->
+  <!--   </inertial> -->
+  <!--   <visual> -->
+  <!--     <origin rpy="0 0 0" xyz="0 0 -0.017"/> -->
+  <!--     <geometry> -->
+  <!--       <box size="0.13 0.044 0.034"/> -->
+  <!--     </geometry> -->
+  <!--   </visual> -->
+  <!-- </link> -->
 </robot>

File: robots/beetle/robots/beetle_fang.urdf.xacro (robot description, xacro)
@@ -77,47 +77,47 @@
   </link>
   <!-- battery -->
-  <joint name="battery1_joint" type="fixed">
-    <parent link="base_link"/>
-    <child link="battery1"/>
-    <origin xyz="0 0.044 0.055" rpy="0 0 0"/>
-    <axis xyz="1 0 0"/>
-  </joint>
-  <link name="battery1">
-    <inertial>
-      <origin xyz="0 0 -0.017" rpy="0 0 0"/>
-      <mass value="0.41"/>
-      <inertia
-          ixx="0.00060259" ixy="0.0" ixz="0.0"
-          iyy="0.00062827" iyz="0.0"
-          izz="0.00010170"/>
-    </inertial>
-    <visual>
-      <origin rpy="0 0 0" xyz="0 0 -0.017"/>
-      <geometry>
-        <box size="0.13 0.044 0.034"/>
-      </geometry>
-    </visual>
-  </link>
-  <joint name="battery2_joint" type="fixed">
-    <parent link="base_link"/>
-    <child link="battery2"/>
-    <origin xyz="0 -0.044 0.055" rpy="0 0 0"/>
-    <axis xyz="1 0 0"/>
-  </joint>
-  <link name="battery2">
-    <inertial>
-      <origin xyz="0 0 -0.017" rpy="0 0 0"/>
-      <mass value="0.41"/>
-      <inertia
-          ixx="0.00060259" ixy="0.0" ixz="0.0"
-          iyy="0.00062827" iyz="0.0"
-          izz="0.00010170"/>
-    </inertial>
-    <visual>
-      <origin rpy="0 0 0" xyz="0 0 -0.017"/>
-      <geometry>
-        <box size="0.13 0.044 0.034"/>
-      </geometry>
-    </visual>
-  </link>
+  <!-- <joint name="battery1_joint" type="fixed"> -->
+  <!--   <parent link="base_link"/> -->
+  <!--   <child link="battery1"/> -->
+  <!--   <origin xyz="0 0.044 0.055" rpy="0 0 0"/> -->
+  <!--   <axis xyz="1 0 0"/> -->
+  <!-- </joint> -->
+  <!-- <link name="battery1"> -->
+  <!--   <inertial> -->
+  <!--     <origin xyz="0 0 -0.017" rpy="0 0 0"/> -->
+  <!--     <mass value="0.41"/> -->
+  <!--     <inertia -->
+  <!--         ixx="0.00060259" ixy="0.0" ixz="0.0" -->
+  <!--         iyy="0.00062827" iyz="0.0" -->
+  <!--         izz="0.00010170"/> -->
+  <!--   </inertial> -->
+  <!--   <visual> -->
+  <!--     <origin rpy="0 0 0" xyz="0 0 -0.017"/> -->
+  <!--     <geometry> -->
+  <!--       <box size="0.13 0.044 0.034"/> -->
+  <!--     </geometry> -->
+  <!--   </visual> -->
+  <!-- </link> -->
+  <!-- <joint name="battery2_joint" type="fixed"> -->
+  <!--   <parent link="base_link"/> -->
+  <!--   <child link="battery2"/> -->
+  <!--   <origin xyz="0 -0.044 0.055" rpy="0 0 0"/> -->
+  <!--   <axis xyz="1 0 0"/> -->
+  <!-- </joint> -->
+  <!-- <link name="battery2"> -->
+  <!--   <inertial> -->
+  <!--     <origin xyz="0 0 -0.017" rpy="0 0 0"/> -->
+  <!--     <mass value="0.41"/> -->
+  <!--     <inertia -->
+  <!--         ixx="0.00060259" ixy="0.0" ixz="0.0" -->
+  <!--         iyy="0.00062827" iyz="0.0" -->
+  <!--         izz="0.00010170"/> -->
+  <!--   </inertial> -->
+  <!--   <visual> -->
+  <!--     <origin rpy="0 0 0" xyz="0 0 -0.017"/> -->
+  <!--     <geometry> -->
+  <!--       <box size="0.13 0.044 0.034"/> -->
+  <!--     </geometry> -->
+  <!--   </visual> -->
+  <!-- </link> -->
 </robot>

File: robots/beetle/urdf/beetle.urdf.xacro (robot description, xacro)
@@ -23,5 +23,6 @@
     <link name="base_link">
       <inertial>
-        <origin xyz="0.0071144 0.0004661 0.1372857" rpy="0 0 0"/>
+        <!-- <origin xyz="0.0071144 0.0004661 0.1372857" rpy="0 0 0"/> -->
+	<origin xyz="-0.009 0.0004661 0.1372857" rpy="0 0 0"/>
         <mass value="2.7703823"/>
         <inertia

Commit message: [Beetle_hyper][urdf] fix the misaligned defination

File: robots/beetle/robots/beetle.urdf.xacro (robot description, xacro)
@@ -13,5 +13,5 @@
     <parent link="base_link"/>
     <child link="dummy_arm"/>
-    <origin xyz="0.22 0 0.1455" rpy="0 0 0"/>
+    <origin xyz="0.239 0 0.0895" rpy="0 0 0"/>
   </joint>
   <link name="dummy_arm">
@@ -80,5 +80,5 @@
     <parent link="base_link"/>
     <child link="battery1"/>
-    <origin xyz="0 0.044 0.055" rpy="0 0 0"/>
+    <origin xyz="0 0.044 -0.01" rpy="0 0 0"/>
     <axis xyz="1 0 0"/>
   </joint>
@@ -102,5 +102,5 @@
     <parent link="base_link"/>
     <child link="battery2"/>
-    <origin xyz="0 -0.044 0.055" rpy="0 0 0"/>
+    <origin xyz="0 -0.044 -0.01" rpy="0 0 0"/>
     <axis xyz="1 0 0"/>
   </joint>

File: robots/beetle/robots/beetle_fang.urdf.xacro (robot description, xacro)
@@ -13,5 +13,5 @@
     <parent link="base_link"/>
     <child link="dummy_arm"/>
-    <origin xyz="0.22 0 0.1455" rpy="0 0 0"/>
+    <origin xyz="0.239 0 0.0895" rpy="0 0 0"/>
   </joint>
   <link name="dummy_arm">
@@ -80,5 +80,5 @@
     <parent link="base_link"/>
     <child link="battery1"/>
-    <origin xyz="0 0.044 0.055" rpy="0 0 0"/>
+    <origin xyz="0 0.044 -0.01" rpy="0 0 0"/>
     <axis xyz="1 0 0"/>
   </joint>
@@ -102,5 +102,5 @@
     <parent link="base_link"/>
     <child link="battery2"/>
-    <origin xyz="0 -0.044 0.055" rpy="0 0 0"/>
+    <origin xyz="0 -0.044 -0.01" rpy="0 0 0"/>
     <axis xyz="1 0 0"/>
   </joint>

File: robots/beetle/urdf/beetle.urdf.xacro (robot description, xacro)
@@ -32,9 +32,9 @@
         <origin xyz="0 0 0" rpy="0 0 3.141592"/>
         <geometry>
-          <mesh filename="package://beetle/urdf/mesh/base_link.dae"/>
+          <mesh filename="package://beetle/urdf/mesh/base_link_hyper.dae"/>
         </geometry>
       </visual>
       <collision>
-        <origin xyz="0 0 0.1205" rpy="0 0 0"/>
+        <origin xyz="0 0 0.0575" rpy="0 0 0"/>
         <geometry>
           <box size="0.52 0.52 0.241"/>
@@ -56,5 +56,5 @@
       <child link="fc"/>
       <parent link="base_link"/>
-      <origin rpy="0 0 0" xyz="0 0 0.12947"/>
+      <origin rpy="0 0 0" xyz="0 0 0.06747"/>
       <axis xyz="0 0 1"/>
     </joint>
@@ -81,8 +81,8 @@
     </xacro:macro>
     ## dummy rotor arms
-    <xacro:dummy_rotor_arm id = "${child1}" x = "0.12129" y="0.12150" z = "0.1185" yaw = "${pi/4.0}"/>
-    <xacro:dummy_rotor_arm id = "${child2}" x = "-0.12129" y="0.12150" z = "0.1185" yaw = "${pi*3.0/4.0}"/>
-    <xacro:dummy_rotor_arm id = "${child3}" x = "-0.12129" y="-0.12150" z = "0.1185" yaw = "${pi*5.0/4.0}"/>
-    <xacro:dummy_rotor_arm id = "${child4}" x = "0.12129" y="-0.12150" z = "0.1185" yaw = "${-pi/4.0}"/>
+    <xacro:dummy_rotor_arm id = "${child1}" x = "0.12129" y="0.12150" z = "0.0555" yaw = "${pi/4.0}"/>
+    <xacro:dummy_rotor_arm id = "${child2}" x = "-0.12129" y="0.12150" z = "0.0555" yaw = "${pi*3.0/4.0}"/>
+    <xacro:dummy_rotor_arm id = "${child3}" x = "-0.12129" y="-0.12150" z = "0.0555" yaw = "${pi*5.0/4.0}"/>
+    <xacro:dummy_rotor_arm id = "${child4}" x = "0.12129" y="-0.12150" z = "0.0555" yaw = "${-pi/4.0}"/>
     ## dummy link for the contact point coordinate
       <link name="contact_point">
@@ -116,5 +116,5 @@
       </inertial>
       <collision>
-        <origin xyz="0.0 0 0" rpy="0 0 0"/>
+        <origin xyz="0.022 0 0" rpy="0 0 0"/>
         <geometry>
           <cylinder radius="0.02" length="0.033"/>

File: robots/beetle/urdf/beetle_fang.urdf.xacro (robot description, xacro)
@@ -32,10 +32,10 @@
         <origin xyz="0 0 0" rpy="0 0 3.141592"/>
         <geometry>
-          <mesh filename="package://beetle/urdf/mesh/base_link.dae"/>
+          <mesh filename="package://beetle/urdf/mesh/base_link_hyper.dae"/>
         </geometry>
       </visual>
       <!-- decompse the collison part for manipulator -->
       <collision>
-        <origin xyz="-0.09 0 0.1205" rpy="0 0 0"/>
+        <origin xyz="-0.09 0 0.0575" rpy="0 0 0"/>
         <geometry>
           <box size="0.34 0.52 0.241"/>
@@ -43,5 +43,5 @@
       </collision>
       <collision>
-        <origin xyz="0.17 0 0.14256" rpy="0 0 0"/>
+        <origin xyz="0.17 0 0.07956" rpy="0 0 0"/>
         <geometry>
           <box size="0.18 0.52 0.19688"/>
@@ -49,5 +49,5 @@
       </collision>
       <collision>
-        <origin xyz="0.17 0.24 0.02206" rpy="0 0 0"/>
+        <origin xyz="0.17 0.24 -0.04094" rpy="0 0 0"/>
         <geometry>
           <box size="0.18 0.040 0.04412"/>
@@ -55,5 +55,5 @@
       </collision>
       <collision>
-        <origin xyz="0.17 -0.24 0.02206" rpy="0 0 0"/>
+        <origin xyz="0.17 -0.24 -0.04094" rpy="0 0 0"/>
         <geometry>
           <box size="0.18 0.040 0.04412"/>
@@ -75,5 +75,5 @@
       <child link="fc"/>
       <parent link="base_link"/>
-      <origin rpy="0 0 0" xyz="0 0 0.12947"/>
+      <origin rpy="0 0 0" xyz="0 0 0.06747"/>
       <axis xyz="0 0 1"/>
     </joint>
@@ -109,5 +109,5 @@
       <parent link="base_link"/>
       <child link="beetle_fang_link"/>
-      <origin xyz="0.246 0 0.0743823" rpy="0 0 0"/>
+      <origin xyz="0.246 0 0.0113823" rpy="0 0 0"/>
     </joint>
     ## rotor arm macro
@@ -133,8 +133,8 @@
     </xacro:macro>
     ## dummy rotor arms
-    <xacro:dummy_rotor_arm id = "${child1}" x = "0.12129" y="0.12150" z = "0.1185" yaw = "${pi/4.0}"/>
-    <xacro:dummy_rotor_arm id = "${child2}" x = "-0.12129" y="0.12150" z = "0.1185" yaw = "${pi*3.0/4.0}"/>
-    <xacro:dummy_rotor_arm id = "${child3}" x = "-0.12129" y="-0.12150" z = "0.1185" yaw = "${pi*5.0/4.0}"/>
-    <xacro:dummy_rotor_arm id = "${child4}" x = "0.12129" y="-0.12150" z = "0.1185" yaw = "${-pi/4.0}"/>
+    <xacro:dummy_rotor_arm id = "${child1}" x = "0.12129" y="0.12150" z = "0.0555" yaw = "${pi/4.0}"/>
+    <xacro:dummy_rotor_arm id = "${child2}" x = "-0.12129" y="0.12150" z = "0.0555" yaw = "${pi*3.0/4.0}"/>
+    <xacro:dummy_rotor_arm id = "${child3}" x = "-0.12129" y="-0.12150" z = "0.0555" yaw = "${pi*5.0/4.0}"/>
+    <xacro:dummy_rotor_arm id = "${child4}" x = "0.12129" y="-0.12150" z = "0.0555" yaw = "${-pi/4.0}"/>
     ## dummy link for the contact point coordinate
       <link name="contact_point">
@@ -168,5 +168,5 @@
       </inertial>
       <collision>
-        <origin xyz="0.0 0 0" rpy="0 0 0"/>
+        <origin xyz="0.022 0 0" rpy="0 0 0"/>
         <geometry>
           <cylinder radius="0.02" length="0.033"/>

File: robots/gimbalrotor/urdf/beetle_hyper/gimbalrotor.urdf.xacro (robot description, xacro)
@@ -36,5 +36,5 @@
       </visual>
       <collision>
-        <origin xyz="0 0 0.053" rpy="0 0 0"/>
+        <origin xyz="0 0 0.0575" rpy="0 0 0"/>
         <geometry>
           <box size="0.52 0.52 0.241"/>
@@ -116,5 +116,5 @@
       </inertial>
       <collision>
-        <origin xyz="0.0 0 0" rpy="0 0 0"/>
+        <origin xyz="0.022 0 0" rpy="0 0 0"/>
         <geometry>
           <cylinder radius="0.02" length="0.033"/>

Commit message: [Beetle][urdf] fix the wrong defination of dummy grasp link to support assemble in gazebo

File: robots/beetle/robots/beetle.urdf.xacro (robot description, xacro)
@@ -13,5 +13,5 @@
     <parent link="base_link"/>
     <child link="dummy_arm"/>
-    <origin xyz="0.239 0 0.0895" rpy="0 0 0"/>
+    <origin xyz="0.22 0 0.0895" rpy="0 0 0"/>
   </joint>
   <link name="dummy_arm">

File: robots/beetle/robots/beetle_fang.urdf.xacro (robot description, xacro)
@@ -13,5 +13,5 @@
     <parent link="base_link"/>
     <child link="dummy_arm"/>
-    <origin xyz="0.239 0 0.0895" rpy="0 0 0"/>
+    <origin xyz="0.22 0 0.0895" rpy="0 0 0"/>
   </joint>
   <link name="dummy_arm">

Commit message: [Beetle_hyper][assemble]modify the assemble function according to the performance on real machine

File: robots/beetle/robots/beetle.urdf.xacro (robot description, xacro)
@@ -77,5 +77,5 @@
   </link>
   <!-- battery -->
-  <joint name="battery1_joint" type="fixed">
+  <!-- <joint name="battery1_joint" type="fixed">
     <parent link="base_link"/>
     <child link="battery1"/>
@@ -121,3 +121,4 @@
     </visual>
   </link>
+   -->
 </robot>

Commit message: [Beetle_hyper][valve roation] adjust valve roation code based on real-world experiment

File: robots/beetle/robots/beetle.urdf.xacro (robot description, xacro)
@@ -77,5 +77,5 @@
   </link>
   <!-- battery -->
-  <!-- <joint name="battery1_joint" type="fixed">
+  <joint name="battery1_joint" type="fixed">
     <parent link="base_link"/>
     <child link="battery1"/>
@@ -121,4 +121,3 @@
     </visual>
   </link>
-   -->
 </robot>
