Commit message: [Beetle_hyper][model] hovering without battery

File: robots/beetle/robots/beetle.urdf.xacro (robot description, xacro)
@@ -77,5 +77,5 @@
   </link>
   <!-- battery -->
-  <joint name="battery1_joint" type="fixed">
+  <!-- <joint name="battery1_joint" type="fixed">
     <parent link="base_link"/>
     <child link="battery1"/>
@@ -120,4 +120,4 @@
       </geometry>
     </visual>
-  </link>
+  </link> -->
 </robot>

File: robots/beetle/robots/beetle_fang.urdf.xacro (robot description, xacro)
@@ -77,5 +77,5 @@
   </link>
   <!-- battery -->
-  <joint name="battery1_joint" type="fixed">
+  <!-- <joint name="battery1_joint" type="fixed">
     <parent link="base_link"/>
     <child link="battery1"/>
@@ -120,4 +120,4 @@
       </geometry>
     </visual>
-  </link>
+  </link> -->
 </robot>

Commit message: [Beetle][bringup] add launch option for battery

File: robots/beetle/robots/beetle.urdf.xacro (robot description, xacro)
@@ -2,4 +2,5 @@
 <robot
     xmlns:xacro="http://www.ros.org/wiki/xacro" name="beetle" >
+  <xacro:arg name="battery" default="false" />
   <xacro:include filename="$(find beetle)/urdf/beetle.urdf.xacro" />
   <xacro:include filename="$(find beetle)/urdf/common.xacro" />
@@ -77,47 +78,49 @@
   </link>
   <!-- battery -->
-  <!-- <joint name="battery1_joint" type="fixed">
-    <parent link="base_link"/>
-    <child link="battery1"/>
-    <origin xyz="0 0.044 -0.01" rpy="0 0 0"/>
-    <axis xyz="1 0 0"/>
-  </joint>
-  <link name="battery1">
-    <inertial>
-      <origin xyz="0 0 -0.017" rpy="0 0 0"/>
-      <mass value="0.41"/>
-      <inertia
-          ixx="0.00060259" ixy="0.0" ixz="0.0"
-          iyy="0.00062827" iyz="0.0"
-          izz="0.00010170"/>
-    </inertial>
-    <visual>
-      <origin rpy="0 0 0" xyz="0 0 -0.017"/>
-      <geometry>
-        <box size="0.13 0.044 0.034"/>
-      </geometry>
-    </visual>
-  </link>
-  <joint name="battery2_joint" type="fixed">
-    <parent link="base_link"/>
-    <child link="battery2"/>
-    <origin xyz="0 -0.044 -0.01" rpy="0 0 0"/>
-    <axis xyz="1 0 0"/>
-  </joint>
-  <link name="battery2">
-    <inertial>
-      <origin xyz="0 0 -0.017" rpy="0 0 0"/>
-      <mass value="0.41"/>
-      <inertia
-          ixx="0.00060259" ixy="0.0" ixz="0.0"
-          iyy="0.00062827" iyz="0.0"
-          izz="0.00010170"/>
-    </inertial>
-    <visual>
-      <origin rpy="0 0 0" xyz="0 0 -0.017"/>
-      <geometry>
-        <box size="0.13 0.044 0.034"/>
-      </geometry>
-    </visual>
-  </link> -->
+  <xacro:if value="$(arg battery)">
+    <joint name="battery1_joint" type="fixed">
+      <parent link="base_link"/>
+      <child link="battery1"/>
+      <origin xyz="0 0.044 -0.01" rpy="0 0 0"/>
+      <axis xyz="1 0 0"/>
+    </joint>
+    <link name="battery1">
+      <inertial>
+        <origin xyz="0 0 -0.017" rpy="0 0 0"/>
+        <mass value="0.41"/>
+        <inertia
+            ixx="0.00060259" ixy="0.0" ixz="0.0"
+            iyy="0.00062827" iyz="0.0"
+            izz="0.00010170"/>
+      </inertial>
+      <visual>
+        <origin rpy="0 0 0" xyz="0 0 -0.017"/>
+        <geometry>
+          <box size="0.13 0.044 0.034"/>
+        </geometry>
+      </visual>
+    </link>
+    <joint name="battery2_joint" type="fixed">
+      <parent link="base_link"/>
+      <child link="battery2"/>
+      <origin xyz="0 -0.044 -0.01" rpy="0 0 0"/>
+      <axis xyz="1 0 0"/>
+    </joint>
+    <link name="battery2">
+      <inertial>
+        <origin xyz="0 0 -0.017" rpy="0 0 0"/>
+        <mass value="0.41"/>
+        <inertia
+            ixx="0.00060259" ixy="0.0" ixz="0.0"
+            iyy="0.00062827" iyz="0.0"
+            izz="0.00010170"/>
+      </inertial>
+      <visual>
+        <origin rpy="0 0 0" xyz="0 0 -0.017"/>
+        <geometry>
+          <box size="0.13 0.044 0.034"/>
+        </geometry>
+      </visual>
+    </link>
+  </xacro:if>
 </robot>

File: robots/beetle/robots/beetle_fang.urdf.xacro (robot description, xacro)
@@ -2,4 +2,5 @@
 <robot
     xmlns:xacro="http://www.ros.org/wiki/xacro" name="beetle" >
+  <xacro:arg name="battery" default="false" />
   <xacro:include filename="$(find beetle)/urdf/beetle_fang.urdf.xacro" />
   <xacro:include filename="$(find beetle)/urdf/common.xacro" />
@@ -77,47 +78,49 @@
   </link>
   <!-- battery -->
-  <!-- <joint name="battery1_joint" type="fixed">
-    <parent link="base_link"/>
-    <child link="battery1"/>
-    <origin xyz="0 0.044 -0.01" rpy="0 0 0"/>
-    <axis xyz="1 0 0"/>
-  </joint>
-  <link name="battery1">
-    <inertial>
-      <origin xyz="0 0 -0.017" rpy="0 0 0"/>
-      <mass value="0.41"/>
-      <inertia
-          ixx="0.00060259" ixy="0.0" ixz="0.0"
-          iyy="0.00062827" iyz="0.0"
-          izz="0.00010170"/>
-    </inertial>
-    <visual>
-      <origin rpy="0 0 0" xyz="0 0 -0.017"/>
-      <geometry>
-        <box size="0.13 0.044 0.034"/>
-      </geometry>
-    </visual>
-  </link>
-  <joint name="battery2_joint" type="fixed">
-    <parent link="base_link"/>
-    <child link="battery2"/>
-    <origin xyz="0 -0.044 -0.01" rpy="0 0 0"/>
-    <axis xyz="1 0 0"/>
-  </joint>
-  <link name="battery2">
-    <inertial>
-      <origin xyz="0 0 -0.017" rpy="0 0 0"/>
-      <mass value="0.41"/>
-      <inertia
-          ixx="0.00060259" ixy="0.0" ixz="0.0"
-          iyy="0.00062827" iyz="0.0"
-          izz="0.00010170"/>
-    </inertial>
-    <visual>
-      <origin rpy="0 0 0" xyz="0 0 -0.017"/>
-      <geometry>
-        <box size="0.13 0.044 0.034"/>
-      </geometry>
-    </visual>
-  </link> -->
+  <xacro:if value="$(arg battery)">
+    <joint name="battery1_joint" type="fixed">
+      <parent link="base_link"/>
+      <child link="battery1"/>
+      <origin xyz="0 0.044 -0.01" rpy="0 0 0"/>
+      <axis xyz="1 0 0"/>
+    </joint>
+    <link name="battery1">
+      <inertial>
+        <origin xyz="0 0 -0.017" rpy="0 0 0"/>
+        <mass value="0.41"/>
+        <inertia
+            ixx="0.00060259" ixy="0.0" ixz="0.0"
+            iyy="0.00062827" iyz="0.0"
+            izz="0.00010170"/>
+      </inertial>
+      <visual>
+        <origin rpy="0 0 0" xyz="0 0 -0.017"/>
+        <geometry>
+          <box size="0.13 0.044 0.034"/>
+        </geometry>
+      </visual>
+    </link>
+    <joint name="battery2_joint" type="fixed">
+      <parent link="base_link"/>
+      <child link="battery2"/>
+      <origin xyz="0 -0.044 -0.01" rpy="0 0 0"/>
+      <axis xyz="1 0 0"/>
+    </joint>
+    <link name="battery2">
+      <inertial>
+        <origin xyz="0 0 -0.017" rpy="0 0 0"/>
+        <mass value="0.41"/>
+        <inertia
+            ixx="0.00060259" ixy="0.0" ixz="0.0"
+            iyy="0.00062827" iyz="0.0"
+            izz="0.00010170"/>
+      </inertial>
+      <visual>
+        <origin rpy="0 0 0" xyz="0 0 -0.017"/>
+        <geometry>
+          <box size="0.13 0.044 0.034"/>
+        </geometry>
+      </visual>
+    </link>
+  </xacro:if>
 </robot>
